Commit message: removed .parts and moved meshes into meshes folder

File: plato-v2/plato_v2.urdf (robot description, URDF)
Before this commit: robot plato2, 9 links, 8 joints
Links:
- link hand_base: geometry collision mesh filename=package://meshes/hand_base_collision.stl; visual mesh filename=package://meshes/hand_base_visual.stl
- link index_distal: geometry collision mesh filename=package://meshes/index_distal_collision.stl; visual mesh filename=package://meshes/index_distal_visual.stl
- link index_proximal: geometry collision mesh filename=package://meshes/index_proximal_collision.stl; visual mesh filename=package://meshes/index_proximal_visual.stl
- link middle_distal: geometry collision mesh filename=package://meshes/middle_distal_collision.stl; visual mesh filename=package://meshes/middle_distal_visual.stl
- link middle_proximal: geometry collision mesh filename=package://meshes/middle_proximal_collision.stl; visual mesh filename=package://meshes/middle_proximal_visual.stl
- link thumb_actuators: geometry collision mesh filename=package://meshes/thumb_actuators_collision.stl; visual mesh filename=package://meshes/thumb_actuators_visual.stl
- link thumb_distal: geometry collision mesh filename=package://meshes/thumb_distal_collision.stl; visual mesh filename=package://meshes/thumb_distal_visual.stl
- link thumb_metacarpal: geometry collision mesh filename=package://meshes/thumb_metacarpal_collision.stl; visual mesh filename=package://meshes/thumb_metacarpal_visual.stl
- link thumb_proximal: geometry collision mesh filename=package://meshes/thumb_proximal_collision.stl; visual mesh filename=package://meshes/thumb_proximal_visual.stl

Commit message: change meshes to https for foxglove

File: plato-v2/plato_v2.urdf (robot description, URDF)
Before this commit: robot plato2, 9 links, 8 joints
Links:
- link hand_base: geometry collision mesh filename=//https://github.com/Aarim02/plato_v2/blob/master/plato-v2/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; visual mesh filename=//https://github.com/Aarim02/plato_v2/blob/master/plato-v2/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
- link index_distal: geometry collision mesh filename=//https://github.com/Aarim02/plato_v2/blob/master/plato-v2/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; visual mesh filename=//https://github.com/Aarim02/plato_v2/blob/master/plato-v2/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
- link index_proximal: geometry collision mesh filename=//https://github.com/Aarim02/plato_v2/blob/master/plato-v2/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; visual mesh filename=//https://github.com/Aarim02/plato_v2/blob/master/plato-v2/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
- link middle_distal: geometry collision mesh filename=//https://github.com/Aarim02/plato_v2/blob/master/plato-v2/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; visual mesh filename=//https://github.com/Aarim02/plato_v2/blob/master/plato-v2/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
- link middle_proximal: geometry collision mesh filename=//https://github.com/Aarim02/plato_v2/blob/master/plato-v2/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; visual mesh filename=//https://github.com/Aarim02/plato_v2/blob/master/plato-v2/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
- link thumb_actuators: geometry collision mesh filename=//https://github.com/Aarim02/plato_v2/blob/master/plato-v2/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; visual mesh filename=//https://github.com/Aarim02/plato_v2/blob/master/plato-v2/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
- link thumb_distal: geometry collision mesh filename=//https://github.com/Aarim02/plato_v2/blob/master/plato-v2/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; visual mesh filename=//https://github.com/Aarim02/plato_v2/blob/master/plato-v2/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
- link thumb_metacarpal: geometry collision mesh filename=//https://github.com/Aarim02/plato_v2/blob/master/plato-v2/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; visual mesh filename=//https://github.com/Aarim02/plato_v2/blob/master/plato-v2/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
- link thumb_proximal: geometry collision mesh filename=//https://github.com/Aarim02/plato_v2/blob/master/plato-v2/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; visual mesh filename=//https://github.com/Aarim02/plato_v2/blob/master/plato-v2/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

Commit message: Changing url

File: plato-v2/plato_v2.urdf (robot description, URDF)
Before this commit: robot plato2, 9 links, 8 joints
Links:
- link hand_base: geometry collision mesh filename=https://github.com/Aarim02/plato_v2/blob/master/plato-v2/me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; visual mesh filename=https://github.com/Aarim02/plato_v2/blob/master/plato-v2/me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
- link index_distal: geometry collision mesh filename=https://github.com/Aarim02/plato_v2/blob/master/plato-v2/me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; visual mesh filename=https://github.com/Aarim02/plato_v2/blob/master/plato-v2/me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
- link index_proximal: geometry collision mesh filename=https://github.com/Aarim02/plato_v2/blob/master/plato-v2/me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; visual mesh filename=https://github.com/Aarim02/plato_v2/blob/master/plato-v2/me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
- link middle_distal: geometry collision mesh filename=https://github.com/Aarim02/plato_v2/blob/master/plato-v2/me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; visual mesh filename=https://github.com/Aarim02/plato_v2/blob/master/plato-v2/me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
- link middle_proximal: geometry collision mesh filename=https://github.com/Aarim02/plato_v2/blob/master/plato-v2/me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; visual mesh filename=https://github.com/Aarim02/plato_v2/blob/master/plato-v2/me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
- link thumb_actuators: geometry collision mesh filename=https://github.com/Aarim02/plato_v2/blob/master/plato-v2/me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; visual mesh filename=https://github.com/Aarim02/plato_v2/blob/master/plato-v2/me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
- link thumb_distal: geometry collision mesh filename=https://github.com/Aarim02/plato_v2/blob/master/plato-v2/me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; visual mesh filename=https://github.com/Aarim02/plato_v2/blob/master/plato-v2/me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
- link thumb_metacarpal: geometry collision mesh filename=https://github.com/Aarim02/plato_v2/blob/master/plato-v2/me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; visual mesh filename=https://github.com/Aarim02/plato_v2/blob/master/plato-v2/me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
- link thumb_proximal: geometry collision mesh filename=https://github.com/Aarim02/plato_v2/blob/master/plato-v2/me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; visual mesh filename=https://github.com/Aarim02/plato_v2/blob/master/plato-v2/me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

Commit message: changed url to raw.github url

File: plato-v2/plato_v2.urdf (robot description, URDF)
Before this commit: robot plato2, 9 links, 8 joints
Links:
- link hand_base: geometry collision mesh filename=https://raw.githubusercontent.com/Aarim02/plato_v2/refs/hea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; visual mesh filename=https://raw.githubusercontent.com/Aarim02/plato_v2/refs/hea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
- link index_distal: geometry collision mesh filename=https://raw.githubusercontent.com/Aarim02/plato_v2/refs/hea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; visual mesh filename=https://raw.githubusercontent.com/Aarim02/plato_v2/refs/hea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
- link index_proximal: geometry collision mesh filename=https://raw.githubusercontent.com/Aarim02/plato_v2/refs/hea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; visual mesh filename=https://raw.githubusercontent.com/Aarim02/plato_v2/refs/hea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
- link middle_distal: geometry collision mesh filename=https://raw.githubusercontent.com/Aarim02/plato_v2/refs/hea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; visual mesh filename=https://raw.githubusercontent.com/Aarim02/plato_v2/refs/hea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
- link middle_proximal: geometry collision mesh filename=https://raw.githubusercontent.com/Aarim02/plato_v2/refs/hea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; visual mesh filename=https://raw.githubusercontent.com/Aarim02/plato_v2/refs/hea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
- link thumb_actuators: geometry collision mesh filename=https://raw.githubusercontent.com/Aarim02/plato_v2/refs/hea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; visual mesh filename=https://raw.githubusercontent.com/Aarim02/plato_v2/refs/hea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
- link thumb_distal: geometry collision mesh filename=https://raw.githubusercontent.com/Aarim02/plato_v2/refs/hea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; visual mesh filename=https://raw.githubusercontent.com/Aarim02/plato_v2/refs/hea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
- link thumb_metacarpal: geometry collision mesh filename=https://raw.githubusercontent.com/Aarim02/plato_v2/refs/hea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; visual mesh filename=https://raw.githubusercontent.com/Aarim02/plato_v2/refs/hea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
- link thumb_proximal: geometry collision mesh filename=https://raw.githubusercontent.com/Aarim02/plato_v2/refs/hea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; visual mesh filename=https://raw.githubusercontent.com/Aarim02/plato_v2/refs/hea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

Commit message: renamed hand_base to base_link

File: plato-v2/plato_v2.urdf (robot description, URDF)
Before this commit: robot plato2, 9 links, 8 joints
Links:
- removed link hand_base
- added link base_link, mass 0.80648485810857573064; collision mesh filename=https://raw.githubusercontent.com/Aarim02/plato_v2/refs/hea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; visual mesh filename=https://raw.githubusercontent.com/Aarim02/plato_v2/refs/hea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
Joints:
- joint joint1: parent hand_base -> base_link
- joint joint5: parent hand_base -> base_link
- joint joint7: parent hand_base -> base_link
